File: StealthBurner.kicad_pcb (KiCad board)
At the start: 2 copper layers, 45 x 31.5 mm, 15 parts, among them J1 PROBE, J2 E-Step, J3 HE, J4 HET, J5 FS, J6 HEF, J7 PCF, J8 NEO, J9 MCU, M1 M3_hole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

Commit message: 更改线路名称
Connections:
- net /V_FAN renamed Vdrive
Changed lines of the file:
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@@
   (net 15 "/DATA")
   (net 16 "/CBT")
-  (net 17 "/V_FAN")
+  (net 17 "Vdrive")
   (net 18 "/P_SIG")
   (net 19 "/FS")
   (footprint "Logos_User:LassiCat_Logo" (layer "F.Cu")
     (at 148.08 104.693435)
+    (attr board_only exclude_from_pos_files exclude_from_bom)
     (fp_text reference "L1" (at 0 -0.5 unlocked) (layer "F.SilkS") hide
       (effects (font (size 1 1) (thickness 0.15)))
@@
     (fp_line (start -1.11 -2.11) (end -2.36 -2.11) (layer "F.Fab") (width 0.1))
     (pad "1" thru_hole roundrect (at 0 0 270) (size 1.2 1.75) (drill 0.75) (layers *.Cu *.Mask) (roundrect_rratio 0.2083333333)
-      (net 17 "/V_FAN") (pinfunction "Pin_1") (pintype "passive"))
+      (net 17 "Vdrive") (pinfunction "Pin_1") (pintype "passive"))
     (pad "2" thru_hole oval (at 2 0 270) (size 1.2 1.75) (drill 0.75) (layers *.Cu *.Mask)
       (net 13 "/HEF") (pinfunction "Pin_2") (pintype "passive"))
@@
       (net 5 "+24V") (pinfunction "Pin_2") (pintype "passive"))
     (pad "3" thru_hole circle (at 6 0 270) (size 1.5 1.5) (drill 1.02) (layers *.Cu *.Mask)
-      (net 17 "/V_FAN") (pinfunction "Pin_3") (pintype "passive"))
+      (net 17 "Vdrive") (pinfunction "Pin_3") (pintype "passive"))
     (pad "4" thru_hole circle (at 9 0 270) (size 1.5 1.5) (drill 1.02) (layers *.Cu *.Mask)
       (net 18 "/P_SIG") (pinfunction "Pin_4") (pintype "passive"))
@@
     (descr "Mounting Hole 3.2mm, no annular, M3")
     (tags "mounting hole 3.2mm no annular m3")
-    (attr exclude_from_pos_files exclude_from_bom)
+    (attr board_only exclude_from_pos_files exclude_from_bom)
     (fp_text reference "M2" (at 0 -4.2) (layer "F.Fab") hide
       (effects (font (size 1 1) (thickness 0.15)))
@@
     (descr "Mounting Hole 3.2mm, no annular, M3")
     (tags "mounting hole 3.2mm no annular m3")
-    (attr exclude_from_pos_files exclude_from_bom)
+    (attr board_only exclude_from_pos_files exclude_from_bom)
     (fp_text reference "M1" (at 0 -4.2) (layer "F.Fab") hide
       (effects (font (size 1 1) (thickness 0.15)))
@@
     (fp_line (start 3.95 2.8) (end 3.95 -1.7) (layer "F.Fab") (width 0.1))
     (pad "1" thru_hole roundrect (at 0 0 270) (size 1.2 1.75) (drill 0.75) (layers *.Cu *.Mask) (roundrect_rratio 0.2083333333)
-      (net 17 "/V_FAN") (pinfunction "Pin_1") (pintype "passive"))
+      (net 17 "Vdrive") (pinfunction "Pin_1") (pintype "passive"))
     (pad "2" thru_hole oval (at 2 0 270) (size 1.2 1.75) (drill 0.75) (layers *.Cu *.Mask)
       (net 14 "/PCF") (pinfunction "Pin_2") (pintype "passive"))
